Commit message: added file that check if optimized trajectory collides with table on which the robot is fixed. Moreover kinematics of UR is derived is analytical form, so it can be used in trajectory optimization in order to stay away from table, however is considerably slows down the optimization. Even on sever with 40 cpus patter search computes it for hours. Moreover, added files for identification of the pendubot.

File: planar2DOF/planar_manip.urdf (robot description, URDF)
Before this commit: robot Planar 2DOF Manipulator, 4 links, 3 joints
Links:
- link link 1: mass 1 -> 0.29; geometry visual cylinder length=0.25 radius=0.1
- link link 2: mass 0.45 -> 0.26; geometry visual cylinder length=0.25 radius=0.1
Joints:
- joint ee_fixed_joint: origin xyz=1 0 0 rpy=0 0 0 -> xyz=0.25 0 0 rpy=0 0 0
- joint joint 2: origin xyz=1 0 0 rpy=0 0 0 -> xyz=0.25 0 0 rpy=0 0 0

Commit message: indeitification of UR is changed and writeen in terms of functions in order to ease comparison of different data and drive gains. Pendubot indentification is changed to include validation with parameters from CAD

File: planar2DOF/planar_manip.urdf (robot description, URDF)
Before this commit: robot Planar 2DOF Manipulator, 4 links, 3 joints
Links:
- link link 1: mass 0.29 -> 1.085

Commit message: second momentum realizability on a ellipsoid is implemented

File: planar2DOF/planar_manip.urdf (robot description, URDF)
Before this commit: robot Planar 2DOF Manipulator, 4 links, 3 joints
Links:
- link link 2: mass 0.26 -> 0.3

Commit message: rewriting code for identification of the pendubot using classes

File: planar2DOF/planar_manip.urdf (robot description, URDF)
Before this commit: robot Planar 2DOF Manipulator, 4 links, 3 joints
Links:
- link link 2: mass 0.3 -> 0.26
